File: PCB/PCB 1.kicad_pcb (KiCad board)
At the start: 2 copper layers, 4 parts

Commit message: update: Update documentatione and PCB
Parts:
- added REF**: ., Crystal:Crystal_AT310_D3.0mm_L10.0mm_Horizontal, F.Cu at (204.1, 64.8)
- added REF**: ., Connector_PinHeader_2.54mm:PinHeader_1x02_P2.54mm_Horizontal, F.Cu at (169.6, 64.9)
- REF**: value SW_PUSH_6mm_H8.5mm -> sw 1
- moved REF** 131.0 mm to (222.3, 54.6), turned to 90 degrees
- moved REF** 107.5 mm to (172.7, 40.2)
- moved REF** 85.1 mm to (214.6, 36.3)
- moved REF** 82.1 mm to (193.0, 58.2), turned to -90 degrees
Routing:
- net (no net): track 413.8 -> 0.00 mm, vias 16 -> 22
Other:
- board text added: "+"
- board text added: "-"
- board text added: "DC"
- board text added: "OLED 64x128 6 pins"
- board text added: "RES"
- board text added: "SCL"
- board text added: "SDA"
